File: PCB/1st Lvl/Schematics.brd (EAGLE design)
At the start: 62 x 62 mm, 55 parts, among them U1 TPS73533, U10 MSP430FR5969V2, U11 SPARKFUN_USD-SOCKETSMD, U12 SN74CB3T1G125_DCK_5, U13 AS3930, U2 BQ24072_RGT_16, U3 BQ27410-G1_DRZ_12, U4 LSM303DLHC, U5 BU4S66G2, U6 L3GD20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

Commit message: Modified 1st lvl schematic, changed gyro to i2c, board still needs update
Connections:
- net GND: now also U6.4
- net GYR_CS: no longer U6.5
- net I2CCLK: now also U6.2
- net I2CDAT: now also U6.3
- net SPI_CLK: no longer U6.2
- net SPI_MISO: no longer U6.4
- net SPI_MOSI: no longer U6.3
- net VCC: now also U6.5
Routing:
- net SPI_MISO: track 68.2 -> 63.9 mm
- net SPI_MOSI: track 68.1 -> 64.6 mm
- net SPI_CLK: track 64.7 -> 62.3 mm
Changed lines of the file:
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@@
 <layer number="13" name="Route13" color="4" fill="5" visible="no" active="no"/>
 <layer number="14" name="Route14" color="1" fill="6" visible="no" active="no"/>
-<layer number="15" name="VCC" color="10" fill="1" visible="yes" active="yes"/>
+<layer number="15" name="VCC" color="10" fill="1" visible="no" active="yes"/>
 <layer number="16" name="Bottom" color="1" fill="1" visible="yes" active="yes"/>
 <layer number="17" name="Pads" color="2" fill="1" visible="yes" active="yes"/>
@@
 <wire x1="44.7686" y1="41.3396" x2="44.7686" y2="40.5776" width="0.254" layer="1"/>
 <wire x1="44.7686" y1="40.5776" x2="44.323" y2="40.132" width="0.254" layer="1"/>
+<contactref element="U6" pad="4"/>
+<wire x1="16.926" y1="25.999" x2="18.151" y2="29.174" width="0" layer="19" extent="1-1"/>
 </signal>
 <signal name="AGND">
@@
 <via x="43.307" y="46.736" extent="1-16" drill="0.6"/>
 <via x="43.307" y="42.799" extent="1-16" drill="0.6"/>
+<contactref element="U6" pad="5"/>
+<wire x1="17.399" y1="30.099" x2="16.926" y2="27.949" width="0" layer="19" extent="1-16"/>
 </signal>
 <signal name="I2CCLK">
@@
 <wire x1="44.9586" y1="42" x2="43.778" y2="42" width="0.254" layer="1"/>
 <wire x1="43.778" y1="42" x2="43.18" y2="41.402" width="0.254" layer="1"/>
+<contactref element="U6" pad="2"/>
+<wire x1="19.451" y1="29.174" x2="30.25" y2="30.5875" width="0" layer="19" extent="1-1"/>
 </signal>
 <signal name="I2CDAT">
@@
 <wire x1="43.18" y1="45.466" x2="43.714" y2="46" width="0.254" layer="1"/>
 <wire x1="43.714" y1="46" x2="44.9586" y2="46" width="0.254" layer="1"/>
+<contactref element="U6" pad="3"/>
+<wire x1="18.801" y1="29.174" x2="30.75" y2="30.5875" width="0" layer="19" extent="1-1"/>
 </signal>
 <signal name="N$18">
@@
 </signal>
 <signal name="SPI_MOSI">
-<contactref element="U6" pad="3"/>
 <contactref element="U13" pad="13"/>
 <contactref element="U9" pad="31"/>
@@
 <wire x1="25.15" y1="39.025" x2="21.447" y2="35.322" width="0.254" layer="1"/>
 <wire x1="21.447" y1="35.322" x2="18.801" y2="32.676" width="0.254" layer="1"/>
-<wire x1="18.801" y1="32.676" x2="18.801" y2="29.174" width="0.254" layer="1"/>
 <via x="21.447" y="35.322" extent="1-16" drill="0.5"/>
 <wire x1="21.447" y1="35.322" x2="25.638" y2="35.322" width="0.254" layer="16"/>
@@
 </signal>
 <signal name="SPI_MISO">
-<contactref element="U6" pad="4"/>
 <contactref element="U13" pad="14"/>
 <contactref element="U9" pad="17"/>
 <wire x1="21.59" y1="36.83" x2="18.151" y2="33.391" width="0.254" layer="1"/>
-<wire x1="18.151" y1="33.391" x2="18.151" y2="29.174" width="0.254" layer="1"/>
 <wire x1="33.75" y1="30.5875" x2="35.306" y2="32.1435" width="0.254" layer="1"/>
 <wire x1="35.306" y1="32.1435" x2="35.306" y2="33.02" width="0.254" layer="1"/>
@@
 </signal>
 <signal name="SPI_CLK">
-<contactref element="U6" pad="2"/>
 <contactref element="U13" pad="12"/>
 <contactref element="U9" pad="29"/>
-<wire x1="19.451" y1="29.174" x2="19.451" y2="31.576" width="0.254" layer="1"/>
 <wire x1="19.451" y1="31.576" x2="20.671" y2="32.796" width="0.254" layer="1"/>
 <wire x1="20.671" y1="32.796" x2="26.025" y2="38.15" width="0.254" layer="1"/>
@@
 </signal>
 <signal name="GYR_CS">
-<contactref element="U6" pad="5"/>
 <wire x1="29.75" y1="23.4125" x2="29.75" y2="22.003" width="0.254" layer="1"/>
 <wire x1="29.75" y1="22.003" x2="26.162" y2="18.415" width="0.254" layer="1"/>
@@
 <via x="15.621" y="27.94" extent="1-16" drill="0.5"/>
 <wire x1="15.621" y1="27.94" x2="16.917" y2="27.94" width="0.254" layer="1"/>
-<wire x1="16.917" y1="27.94" x2="16.926" y2="27.949" width="0.254" layer="1"/>
 <contactref element="U10" pad="4"/>
 <wire x1="26.162" y1="18.415" x2="24.638" y2="18.415" width="0.254" layer="1"/>
